File: Final_project_rbree.kicad_pcb (KiCad board)
At the start: 2 copper layers, 100 x 60 mm, 44 parts, among them J1 Conn_01x02_Pin, J2 Conn_01x02_Pin, Q1 MMBT3904, Q2 AO3401A, U1 TL431, U2 LTV-817, U3 B1212, U4 2N7002, U7 NE555

Commit message: Add files via upload
Parts:
- added H1: MountingHole, MountingHole:MountingHole_3.2mm_M3, F.Cu at (80.0, 55.0)
- added H2: MountingHole, MountingHole:MountingHole_3.2mm_M3, F.Cu at (80.0, 106.0)
- added H3: MountingHole, MountingHole:MountingHole_3.2mm_M3, F.Cu at (170.0, 55.0)
- added H4: MountingHole, MountingHole:MountingHole_3.2mm_M3, F.Cu at (170.0, 106.0)
- D3: footprint LED_SMD:LED_Cree-XP -> LED_THT:LED_D8.0mm
- moved D2 11.2 mm to (147.1, 93.3), turned to -90 degrees
- moved Conn_01x1 7.80 mm to (151.5, 94.9)
- moved J2 6.50 mm to (88.5, 57.3)
- moved J1 5.23 mm to (80.7, 89.6)
- moved F1 2.79 mm to (89.1, 101.5)
- moved R3 2.10 mm to (89.1, 95.5)
- moved R5 1.40 mm to (89.1, 89.6)
- moved D3 1.12 mm to (164.2, 77.5)
- moved R6 0.70 mm to (89.1, 83.6)
- moved R19 0.60 mm to (169.0, 76.1)
Routing:
- net VCC: track 136.1 -> 116.7 mm
- net GLV+: track 16.0 -> 4.59 mm
- net /RED+: track 22.8 -> 14.4 mm
- net GND: track 128.7 -> 132.3 mm
- net Net-(D3-K): track 3.94 -> 5.64 mm
- net +12V: track 49.2 -> 47.7 mm
- net Net-(J1-Pin_2): track 9.96 -> 11.0 mm
- net Net-(R5-Pad2): track 3.73 -> 3.03 mm
- net Net-(F1-Pad1): track 3.79 -> 3.09 mm
- net Net-(R3-Pad2): track 3.73 -> 3.03 mm
- net Net-(R6-Pad1): track 3.73 -> 3.05 mm
Other:
- outline, holes or cut-outs redrawn

Commit message: Add files via upload
Parts:
- D1: footprint Diode_THT:D_DO-35_SOD27_P7.62mm_Horizontal -> Diode_SMD:D_1206_3216Metric
- U1: footprint Package_TO_SOT_THT:TO-92Flat -> Package_TO_SOT_SMD:SOT-89-3
- moved R19 11.1 mm to (167.7, 65.0)
- moved R21 11.1 mm to (172.0, 62.1)
- moved Q2 7.88 mm to (158.3, 82.1)
- moved R20 7.06 mm to (163.5, 65.0), turned to 90 degrees
- moved D3 4.84 mm to (167.7, 74.2)
- moved D1 4.83 mm to (81.5, 73.5)
- moved R18 1.62 mm to (153.6, 64.1), turned to -90 degrees
- moved R15 1.55 mm to (147.5, 63.5), turned to 180 degrees
- moved C6 1.43 mm to (156.0, 71.7)
- moved U1 1.29 mm to (100.5, 92.6), turned to 90 degrees
- moved D2 0.39 mm to (147.1, 92.9)
- turned C4 to -90 degrees
Routing:
- net Net-(Q1-C): track 33.5 -> 42.1 mm
- net VCC: track 116.7 -> 109.1 mm
- net GND: track 132.3 -> 135.0 mm, vias 1 -> 2
- net Net-(D3-K): track 5.64 -> 7.74 mm
- net Net-(U7-Q): track 7.41 -> 5.40 mm
- net /RED+: track 14.4 -> 12.4 mm
- net Net-(U4-D): track 6.16 -> 8.13 mm
- net Net-(Q1-B): track 2.15 -> 3.86 mm
- net /Vref: track 30.0 -> 28.6 mm
- net Net-(U1-REF): track 7.07 -> 5.94 mm
- net /Vin: track 25.9 -> 25.4 mm

Commit message: Add files via upload
Parts:
- moved J2 11.5 mm to (80.7, 65.8), turned to -90 degrees
- moved D1 8.00 mm to (89.1, 71.2)
- moved R9 7.69 mm to (90.6, 65.8)
- moved R12 7.69 mm to (103.7, 65.8)
- moved R8 7.69 mm to (97.2, 65.8)
- moved R10 4.12 mm to (100.1, 69.8)
- moved R11 3.65 mm to (105.0, 79.0)
- moved C1 3.12 mm to (103.5, 88.2)
- moved C2 2.09 mm to (105.0, 71.3)
- moved LM1 2.01 mm to (112.6, 70.5)
- moved U1 0.42 mm to (100.9, 92.6)
- moved C6 0.30 mm to (155.7, 71.7)
Routing:
- net GND: track 135.0 -> 119.9 mm, vias 2 -> 3
- net Net-(LM1-Pad7): track 31.6 -> 23.9 mm
- net /Vref: track 28.6 -> 22.2 mm
- net Net-(LM1-+): track 12.4 -> 8.48 mm
- net /Vin: track 25.4 -> 21.9 mm
- net Net-(LM1--): track 9.32 -> 10.6 mm

Commit message: Add files via upload
Parts:
- C1, C2, C3, C4, C5, C6, C7, C8: footprint Capacitor_SMD:C_1206_3216Metric -> Capacitor_SMD:C_1206_3216Metric_Pad1.33x1.80mm_HandSolder
- D1: footprint Diode_SMD:D_1206_3216Metric -> Diode_SMD:D_SMA_Handsoldering
- D2: footprint Diode_SMD:D_SMA -> Diode_SMD:D_SMA_Handsoldering
- D3: footprint LED_THT:LED_D8.0mm -> LED_THT:LED_D10.0mm
- Q1, Q2, U4: footprint Package_TO_SOT_SMD:SOT-23 -> Package_TO_SOT_SMD:SOT-23_Handsoldering
- R1, R10, R11, R12, R13, R14, R15, R16, R17, R18, R19, R2, R20, R21, R3, R4, R5, R6, R7, R8, R9: footprint Resistor_SMD:R_1206_3216Metric -> Resistor_SMD:R_1206_3216Metric_Pad1.30x1.75mm_HandSolder
- U2: footprint Package_DIP:DIP-4_W7.62mm -> Package_DIP:SMDIP-4_W9.53mm
- moved C5 8.80 mm to (139.9, 90.1), turned to -90 degrees
- moved R13 4.78 mm to (118.9, 70.4), turned to 90 degrees
- moved U2 4.02 mm to (126.7, 64.8)
- moved D1 3.96 mm to (92.8, 72.7), turned to -90 degrees
- moved C4 2.96 mm to (113.7, 98.9), turned to 90 degrees
- moved D2 2.69 mm to (144.5, 92.4)
- moved D3 0.78 mm to (167.1, 73.8)
- moved Q2 0.56 mm to (158.3, 82.6)
Routing:
- net GND: track 119.9 -> 115.1 mm, vias 3 -> 4
- net +12V: track 47.9 -> 44.4 mm
- net Net-(R13-Pad2): track 4.63 -> 7.86 mm
- net GLV+: track 4.43 -> 7.07 mm
- net /RED+: track 12.4 -> 11.3 mm
- net Net-(U4-G): track 15.7 -> 14.7 mm
- net VCC: track 109.1 -> 110.0 mm
- net Net-(LM1-Pad7): track 23.9 -> 23.1 mm, vias 2 -> 3
