File: Final_project_rbree.kicad_pcb (KiCad board)
At the start: 2 copper layers, 100 x 60 mm, 48 parts, among them J1 Conn_01x02_Pin, J2 Conn_01x02_Pin, Q1 MMBT3904, Q2 AO3401A, U1 TL431, U2 LTV-817, U3 B1212, U4 2N7002, U7 NE555

Commit message: Add files via upload
Parts:
- moved D3 1.74 mm to (167.7, 75.4)
- moved R14 1.19 mm to (137.9, 69.2)
- moved Conn_01x1 1.16 mm to (150.4, 94.9)
- moved Q1 1.01 mm to (157.4, 63.5)
- moved R20 1.01 mm to (162.5, 65.0)
- moved R18 1.01 mm to (152.6, 64.1)
- moved C5 0.81 mm to (139.1, 89.9), turned to 0 degrees
- moved C6 0.50 mm to (155.2, 71.7)
- moved D1 0.38 mm to (92.8, 72.3)
- moved R8 0.17 mm to (97.0, 65.8)
- moved R21 0.16 mm to (172.0, 61.9)
- moved R15 0.09 mm to (147.4, 63.5)
Routing:
- net VCC: track 110.0 -> 107.8 mm
- net GND: track 115.1 -> 113.8 mm
- net Net-(D3-K): track 7.58 -> 8.81 mm
- net GLV+: track 7.07 -> 5.91 mm
- net Net-(U7-Q): track 5.40 -> 4.48 mm
- net Net-(Q1-B): track 3.86 -> 3.30 mm
- net +12V: track 44.4 -> 44.9 mm
- net Net-(Q1-C): track 42.0 -> 42.5 mm
